File: SUN6502.kicad_sch (KiCad schematic)
At the start: 52 parts, among them J1 Barrel_Jack_MountingPin, J2 6-5530843-5, J3 6-5530843-5, J4 DE9_Socket, SW1 RESET, SW2 Power Switch, U1 W65C02SxP, U10 MAX232, U11 74LS00, U2 KM62256CLP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

Commit message: updates, board works
Connections:
- net GND: now also U11.10, U11.12, U11.13, U11.9, U5.13 (A1), U5.14 (A0), U5.15 (E), U8.16 (~{DCD}), U8.17 (~{DSR}), U8.9 (~{CTS})
- no-connect marks 103 -> 93
Other:
- moved on the sheet: U5B
